File: imsensor-v01.sch (EAGLE design)
At the start: 13 parts, among them J1-A3 PJ-313-SPAD, J2-A2 PJ-313-SPAD, J3-A1 PJ-313-SPAD, J4-D3 PJ-313-SPAD, J5-D5 PJ-313-SPAD, J6-D6 PJ-313-SPAD, U1 ARDUINO_SHIELDNO_SILK

Commit message: IM Sensor Node v0.2
Parts:
- added D2-3, DOUT: (no value), SparkFun-Connectors:M03PTH
Connections:
- new net N$13: D2-3.1, J4-D3.SHIELD1, U1.*D3
- new net N$14: D2-3.3, U1.D2
- net GND: now also DOUT.2
- net N$8: now also D2-3.2, DOUT.3; no longer J4-D3.SHIELD1, U1.*D3
- net VCC: now also DOUT.1
Changed lines of the file:
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@@
 <part name="SUPPLY3" library="SparkFun-Aesthetics" deviceset="VCC" device=""/>
 <part name="CURRENT" library="SparkFun-Connectors" deviceset="M02" device="PTH"/>
+<part name="DOUT" library="SparkFun-Connectors" deviceset="M03" device="PTH"/>
+<part name="SUPPLY5" library="SparkFun-Aesthetics" deviceset="VCC" device=""/>
+<part name="GND5" library="SparkFun-Aesthetics" deviceset="GND" device=""/>
+<part name="D2-3" library="SparkFun-Connectors" deviceset="M03" device="PTH"/>
 </parts>
 <sheets>
@@
 <attribute name="NAME" x="65.278" y="55.88" size="1.778" layer="95" rot="R90"/>
 </instance>
+<instance part="DOUT" gate="G$1" x="45.72" y="127" rot="R270"/>
+<instance part="SUPPLY5" gate="G$1" x="38.1" y="111.76" rot="R90"/>
+<instance part="GND5" gate="1" x="45.72" y="109.22"/>
+<instance part="D2-3" gate="G$1" x="63.5" y="127" rot="R270"/>
 </instances>
 <busses>
@@
 <pinref part="GND4" gate="1" pin="GND"/>
 </segment>
+<segment>
+<pinref part="DOUT" gate="G$1" pin="2"/>
+<wire x1="45.72" y1="119.38" x2="45.72" y2="111.76" width="0.1524" layer="91"/>
+<pinref part="GND5" gate="1" pin="GND"/>
+</segment>
 </net>
 <net name="VCC" class="0">
@@
 <pinref part="SUPPLY3" gate="G$1" pin="VCC"/>
 </segment>
+<segment>
+<pinref part="SUPPLY5" gate="G$1" pin="VCC"/>
+<pinref part="DOUT" gate="G$1" pin="1"/>
+<wire x1="38.1" y1="111.76" x2="43.18" y2="111.76" width="0.1524" layer="91"/>
+<wire x1="43.18" y1="111.76" x2="43.18" y2="119.38" width="0.1524" layer="91"/>
+</segment>
 </net>
 <net name="N$9" class="0">
@@
 <pinref part="J5-D5" gate="G$1" pin="L2"/>
 <wire x1="134.62" y1="60.96" x2="139.7" y2="60.96" width="0.1524" layer="91"/>
-</segment>
-</net>
-<net name="N$8" class="0">
-<segment>
-<wire x1="127" y1="99.06" x2="127" y2="81.28" width="0.1524" layer="91"/>
-<pinref part="J4-D3" gate="G$1" pin="SHIELD1"/>
-<wire x1="139.7" y1="81.28" x2="127" y2="81.28" width="0.1524" layer="91"/>
-<wire x1="127" y1="99.06" x2="78.74" y2="99.06" width="0.1524" layer="91"/>
-<pinref part="U1" gate="G$1" pin="*D3"/>
-<wire x1="78.74" y1="116.84" x2="81.28" y2="116.84" width="0.1524" layer="91"/>
-<wire x1="78.74" y1="99.06" x2="78.74" y2="116.84" width="0.1524" layer="91"/>
 </segment>
 </net>
@@
 </segment>
 </net>
+<net name="N$14" class="0">
+<segment>
+<pinref part="D2-3" gate="G$1" pin="3"/>
+<wire x1="66.04" y1="119.38" x2="66.04" y2="114.3" width="0.1524" layer="91"/>
+<pinref part="U1" gate="G$1" pin="D2"/>
+<wire x1="66.04" y1="114.3" x2="81.28" y2="114.3" width="0.1524" layer="91"/>
+</segment>
+</net>
+<net name="N$13" class="0">
+<segment>
+<wire x1="127" y1="99.06" x2="127" y2="81.28" width="0.1524" layer="91"/>
+<pinref part="J4-D3" gate="G$1" pin="SHIELD1"/>
+<wire x1="139.7" y1="81.28" x2="127" y2="81.28" width="0.1524" layer="91"/>
+<wire x1="127" y1="99.06" x2="78.74" y2="99.06" width="0.1524" layer="91"/>
+<wire x1="78.74" y1="99.06" x2="78.74" y2="116.84" width="0.1524" layer="91"/>
+<pinref part="U1" gate="G$1" pin="*D3"/>
+<wire x1="81.28" y1="116.84" x2="78.74" y2="116.84" width="0.1524" layer="91"/>
+<pinref part="D2-3" gate="G$1" pin="1"/>
+<wire x1="78.74" y1="116.84" x2="60.96" y2="116.84" width="0.1524" layer="91"/>
+<wire x1="60.96" y1="119.38" x2="60.96" y2="116.84" width="0.1524" layer="91"/>
+<junction x="78.74" y="116.84"/>
+</segment>
+</net>
+<net name="N$8" class="0">
+<segment>
+<pinref part="D2-3" gate="G$1" pin="2"/>
+<wire x1="63.5" y1="111.76" x2="63.5" y2="119.38" width="0.1524" layer="91"/>
+<pinref part="DOUT" gate="G$1" pin="3"/>
+<wire x1="48.26" y1="119.38" x2="48.26" y2="111.76" width="0.1524" layer="91"/>
+<wire x1="48.26" y1="111.76" x2="63.5" y2="111.76" width="0.1524" layer="91"/>
+</segment>
+</net>
