File: imsensor-esp-v01.brd (EAGLE design)
At the start: 53 x 75.2 mm, 39 parts, among them J1-A2 PJ-313-SPAD, J2-A3 PJ-313-SPAD, J3-A4 PJ-313-SPAD, J4-A5 PJ-313-SPAD, J5-D1 PJ-313-SPAD, J6-D6 PJ-313-SPAD, J7-D5 PJ-313-SPAD, J8-D3 PJ-313-SPAD, Q1 MOSFET-NCHANNEL2N7000, Q2 MOSFET-NCHANNEL2N7000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

Commit message: Finished first layout
Parts:
- added C4: 100nF, SparkFun-Capacitors:CAP-PTH-SMALL
- added C5: 10uF, SparkFun-Capacitors:CPOL-RADIAL-10UF-25V
- added U2: 78D33, salvador-parts-imported:TO220-IGO
- C1, C2: value (none) -> 10uF
- C3: value (none) -> 100nF
- CURRENT0, CURRENT1, PROG: value (none) -> 2PIN
- D1, D2: device adafruit:DO35-7 -> adafruit:DO41-7
- D2-3, DOUT, ESP-PROG: value (none) -> 3PIN
- S1: device SparkFun-Electromechanical:TACTILE-PTH -> salvador-parts-imported2:TACTILE-PTH
- moved ESP-PROG 86.3 mm to (7.75, 63.6), turned to 270 degrees
- moved D1 82.7 mm to (1.65, 65.0), turned to 270 degrees
- moved D2 78.1 mm to (4.45, 65.0), turned to 90 degrees
- moved C3 73.9 mm to (9.65, 69.1), turned to 180 degrees
- moved Q2 57.1 mm to (16.8, 39.8), turned to 0 degrees
- moved Q1 52.8 mm to (23.1, 38.1), turned to 0 degrees
- moved R11 48.0 mm to (15.5, 29.1), turned to 270 degrees
- moved R12 47.2 mm to (18.0, 30.4), turned to 270 degrees
- moved R9 41.8 mm to (21.8, 29.1), turned to 270 degrees
- moved R10 40.1 mm to (24.4, 29.1), turned to 270 degrees
- moved J1-A2 9.91 mm to (7.62, 83.1)
- moved J2-A3 9.91 mm to (20.3, 83.1)
- moved J3-A4 9.91 mm to (33.0, 83.1)
- moved J4-A5 9.91 mm to (45.7, 83.1)
- moved S1 7.15 mm to (18.5, 62.2)
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- renumbered J5-D1 to J5-D9
Connections:
- net 3.3V: now also C5.1, U2.OUT
- net GND: now also C4.2, C5.2, S1.2, U2.GND
- net VCC: now also C4.1, U2.IN
Routing:
- net VCC: track 110.3 -> 173.6 mm
- net TX: track 0.00 -> 59.1 mm
- net RX: track 0.00 -> 56.4 mm
- net 3.3V: track 27.7 -> 83.4 mm
- net N$22: track 16.6 -> 70.4 mm
- net GND: track 249.7 -> 301.6 mm
- net N$21: track 0.00 -> 39.4 mm
- net N$18: track 0.00 -> 31.9 mm
- net N$25: track 24.8 -> 52.2 mm
- net N$5: track 54.9 -> 65.1 mm
- net N$4: track 42.3 -> 52.2 mm
- net N$15: track 17.6 -> 27.5 mm
- net N$3: track 28.0 -> 37.9 mm
- net U$1: track 0.00 -> 5.49 mm
- net DTR: track 0.00 -> 5.11 mm
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Other:
- board size 53 x 75.2 mm -> 53.1 x 84.2 mm
