File: imsensor-esp-v01.sch (EAGLE design)
At the start: 39 parts, among them J1-A2 PJ-313-SPAD, J2-A3 PJ-313-SPAD, J3-A4 PJ-313-SPAD, J4-A5 PJ-313-SPAD, J5-D1 PJ-313-SPAD, J6-D6 PJ-313-SPAD, J7-D5 PJ-313-SPAD, J8-D3 PJ-313-SPAD, Q1 MOSFET-NCHANNEL2N7000, Q2 MOSFET-NCHANNEL2N7000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

Commit message: Finished first layout
Parts:
- added C4: 100nF, SparkFun-Capacitors:CAPPTH
- added C5: 10uF, SparkFun-Capacitors:10UF-25V-20%(PTH)
- added U2: 78D33, salvador-parts-imported:V_REG_78XXSINK
- C1, C2: value (none) -> 10uF
- C3: value (none) -> 100nF
- CURRENT0, CURRENT1, PROG: value (none) -> 2PIN
- D1, D2: device adafruit:SCHOTTKY-DIODEDO35-7 -> adafruit:SCHOTTKY-DIODEDO41-7
- D2-3, DOUT, ESP-PROG: value (none) -> 3PIN
- S1: device SparkFun-Electromechanical:SWITCH-MOMENTARY-2PTH -> salvador-parts-imported2:SWITCH-MOMENTARY-2PTH
- renumbered J5-D1 to J5-D9
Connections:
- net 3.3V: now also C5.+, U2.OUT
- net GND: now also C4.2, C5.-, S1.P$1, U2.GND
- net VCC: now also C4.1, U2.IN
Changed lines of the file:
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@@
 <part name="R3" library="resistor" deviceset="R-US_" device="0207/10" value="470K"/>
 <part name="R4" library="resistor" deviceset="R-US_" device="0207/10" value="470K"/>
-<part name="C1" library="SparkFun-Capacitors" deviceset="10UF-25V-20%(PTH)" device=""/>
+<part name="C1" library="SparkFun-Capacitors" deviceset="10UF-25V-20%(PTH)" device="" value="10uF"/>
 <part name="GND3" library="SparkFun-Aesthetics" deviceset="GND" device=""/>
 <part name="GND4" library="SparkFun-Aesthetics" deviceset="GND" device=""/>
 <part name="SUPPLY3" library="SparkFun-Aesthetics" deviceset="VCC" device=""/>
-<part name="CURRENT1" library="SparkFun-Connectors" deviceset="M02" device="PTH"/>
-<part name="DOUT" library="SparkFun-Connectors" deviceset="M03" device="PTH"/>
+<part name="CURRENT1" library="SparkFun-Connectors" deviceset="M02" device="PTH" value="2PIN"/>
+<part name="DOUT" library="SparkFun-Connectors" deviceset="M03" device="PTH" value="3PIN"/>
 <part name="SUPPLY5" library="SparkFun-Aesthetics" deviceset="VCC" device=""/>
 <part name="GND5" library="SparkFun-Aesthetics" deviceset="GND" device=""/>
-<part name="D2-3" library="SparkFun-Connectors" deviceset="M03" device="PTH"/>
+<part name="D2-3" library="SparkFun-Connectors" deviceset="M03" device="PTH" value="3PIN"/>
 <part name="J4-A5" library="salvador-parts" deviceset="PJ-313-SPAD" device="" value="PJ-313-SPAD"/>
-<part name="J5-D1" library="salvador-parts" deviceset="PJ-313-SPAD" device="" value="PJ-313-SPAD"/>
+<part name="J5-D9" library="salvador-parts" deviceset="PJ-313-SPAD" device="" value="PJ-313-SPAD"/>
 <part name="R5" library="resistor" deviceset="R-US_" device="0207/10" value="64"/>
 <part name="R6" library="resistor" deviceset="R-US_" device="0207/10" value="82"/>
 <part name="R7" library="resistor" deviceset="R-US_" device="0207/10" value="470K"/>
 <part name="R8" library="resistor" deviceset="R-US_" device="0207/10" value="470K"/>
-<part name="C2" library="SparkFun-Capacitors" deviceset="10UF-25V-20%(PTH)" device=""/>
+<part name="C2" library="SparkFun-Capacitors" deviceset="10UF-25V-20%(PTH)" device="" value="10uF"/>
 <part name="GND6" library="SparkFun-Aesthetics" deviceset="GND" device=""/>
 <part name="GND7" library="SparkFun-Aesthetics" deviceset="GND" device=""/>
 <part name="SUPPLY6" library="SparkFun-Aesthetics" deviceset="VCC" device=""/>
-<part name="CURRENT0" library="SparkFun-Connectors" deviceset="M02" device="PTH"/>
+<part name="CURRENT0" library="SparkFun-Connectors" deviceset="M02" device="PTH" value="2PIN"/>
 <part name="ESP" library="esp8266-modules" deviceset="ESP01" device=""/>
 <part name="R9" library="resistor" deviceset="R-US_" device="0207/10" value="2.2K"/>
@@
 <part name="R15" library="resistor" deviceset="R-US_" device="0207/10" value="10K"/>
 <part name="SUPPLY14" library="SparkFun-Aesthetics" deviceset="3.3V" device=""/>
-<part name="C3" library="SparkFun-Capacitors" deviceset="CAP" device="PTH"/>
-<part name="D1" library="adafruit" deviceset="SCHOTTKY-DIODE" device="DO35-7" value="1N5817"/>
-<part name="ESP-PROG" library="SparkFun-Connectors" deviceset="M03" device="PTH"/>
-<part name="D2" library="adafruit" deviceset="SCHOTTKY-DIODE" device="DO35-7" value="1N5817"/>
-<part name="PROG" library="SparkFun-Connectors" deviceset="M02" device="PTH"/>
+<part name="C3" library="SparkFun-Capacitors" deviceset="CAP" device="PTH" value="100nF"/>
+<part name="D1" library="adafruit" deviceset="SCHOTTKY-DIODE" device="DO41-7" value="1N5817"/>
+<part name="ESP-PROG" library="SparkFun-Connectors" deviceset="M03" device="PTH" value="3PIN"/>
+<part name="D2" library="adafruit" deviceset="SCHOTTKY-DIODE" device="DO41-7" value="1N5817"/>
+<part name="PROG" library="SparkFun-Connectors" deviceset="M02" device="PTH" value="2PIN"/>
 <part name="GND9" library="SparkFun-Aesthetics" deviceset="GND" device=""/>
-<part name="S1" library="SparkFun-Electromechanical" deviceset="SWITCH-MOMENTARY-2" device="PTH"/>
+<part name="S1" library="salvador-parts-imported2" deviceset="SWITCH-MOMENTARY-2" device="PTH"/>
 <part name="GND10" library="SparkFun-Aesthetics" deviceset="GND" device=""/>
+<part name="U2" library="salvador-parts-imported" deviceset="V_REG_78XX" device="SINK" value="78D33"/>
+<part name="C4" library="SparkFun-Capacitors" deviceset="CAP" device="PTH" value="100nF"/>
+<part name="C5" library="SparkFun-Capacitors" deviceset="10UF-25V-20%(PTH)" device="" value="10uF"/>
+<part name="GND11" library="SparkFun-Aesthetics" deviceset="GND" device=""/>
+<part name="GND12" library="SparkFun-Aesthetics" deviceset="GND" device=""/>
+<part name="GND13" library="SparkFun-Aesthetics" deviceset="GND" device=""/>
+<part name="SUPPLY15" library="SparkFun-Aesthetics" deviceset="3.3V" device=""/>
+<part name="SUPPLY16" library="SparkFun-Aesthetics" deviceset="VCC" device=""/>
 </parts>
 <sheets>
@@
 <attribute name="VALUE" x="238.76" y="144.78" size="2.1844" layer="96" font="vector" rot="MR0" display="off"/>
 </instance>
-<instance part="J5-D1" gate="G$1" x="233.68" y="30.48" smashed="yes" rot="MR0">
+<instance part="J5-D9" gate="G$1" x="233.68" y="30.48" smashed="yes" rot="MR0">
 <attribute name="NAME" x="238.76" y="35.56" size="2.1844" layer="95" font="vector" rot="MR0"/>
 <attribute name="VALUE" x="238.76" y="22.86" size="2.1844" layer="96" font="vector" rot="MR0" display="off"/>
@@
 <attribute name="VALUE" x="81.28" y="66.04" size="1.778" layer="96" display="off"/>
 </instance>
-<instance part="GND10" gate="1" x="73.66" y="68.58" rot="R270"/>
+<instance part="GND10" gate="1" x="71.12" y="68.58" rot="R270"/>
+<instance part="U2" gate="G$1" x="48.26" y="152.4"/>
+<instance part="C4" gate="G$1" x="33.02" y="144.78"/>
+<instance part="C5" gate="G$1" x="63.5" y="147.32"/>
+<instance part="GND11" gate="1" x="48.26" y="137.16"/>
+<instance part="GND12" gate="1" x="33.02" y="137.16"/>
+<instance part="GND13" gate="1" x="63.5" y="137.16"/>
+<instance part="SUPPLY15" gate="G$1" x="71.12" y="152.4" rot="R270"/>
+<instance part="SUPPLY16" gate="G$1" x="25.4" y="152.4" rot="R90"/>
 </instances>
 <busses>
@@
 <wire x1="218.44" y1="48.26" x2="218.44" y2="30.48" width="0.1524" layer="91"/>
 <junction x="218.44" y="48.26"/>
-<pinref part="J5-D1" gate="G$1" pin="R"/>
+<pinref part="J5-D9" gate="G$1" pin="R"/>
 <wire x1="218.44" y1="30.48" x2="226.06" y2="30.48" width="0.1524" layer="91"/>
 </segment>
@@
 <wire x1="78.74" y1="68.58" x2="76.2" y2="68.58" width="0.1524" layer="91"/>
 <pinref part="GND10" gate="1" pin="GND"/>
+<pinref part="S1" gate="G$1" pin="P$1"/>
+<wire x1="76.2" y1="68.58" x2="73.66" y2="68.58" width="0.1524" layer="91"/>
+<wire x1="78.74" y1="66.04" x2="76.2" y2="66.04" width="0.1524" layer="91"/>
+<wire x1="76.2" y1="66.04" x2="76.2" y2="68.58" width="0.1524" layer="91"/>
+<junction x="76.2" y="68.58"/>
+</segment>
+<segment>
+<pinref part="U2" gate="G$1" pin="GND"/>
+<wire x1="48.26" y1="144.78" x2="48.26" y2="139.7" width="0.1524" layer="91"/>
+<pinref part="GND11" gate="1" pin="GND"/>
+</segment>
+<segment>
+<pinref part="C4" gate="G$1" pin="2"/>
+<pinref part="GND12" gate="1" pin="GND"/>
+<wire x1="33.02" y1="142.24" x2="33.02" y2="139.7" width="0.1524" layer="91"/>
+</segment>
+<segment>
+<pinref part="C5" gate="G$1" pin="-"/>
+<pinref part="GND13" gate="1" pin="GND"/>
+<wire x1="63.5" y1="142.24" x2="63.5" y2="139.7" width="0.1524" layer="91"/>
 </segment>
 </net>
@@
 <wire x1="93.98" y1="111.76" x2="93.98" y2="116.84" width="0.1524" layer="91"/>
 <pinref part="SUPPLY8" gate="G$1" pin="VCC"/>
+</segment>
+<segment>
+<pinref part="U2" gate="G$1" pin="IN"/>
+<pinref part="C4" gate="G$1" pin="1"/>
+<wire x1="40.64" y1="152.4" x2="33.02" y2="152.4" width="0.1524" layer="91"/>
+<wire x1="33.02" y1="152.4" x2="33.02" y2="149.86" width="0.1524" layer="91"/>
+<wire x1="33.02" y1="152.4" x2="25.4" y2="152.4" width="0.1524" layer="91"/>
+<junction x="33.02" y="152.4"/>
+<pinref part="SUPPLY16" gate="G$1" pin="VCC"/>
 </segment>
 </net>
@@
 <wire x1="226.06" y1="50.8" x2="220.98" y2="50.8" width="0.1524" layer="91"/>
 <wire x1="220.98" y1="50.8" x2="220.98" y2="25.4" width="0.1524" layer="91"/>
-<pinref part="J5-D1" gate="G$1" pin="L2"/>
+<pinref part="J5-D9" gate="G$1" pin="L2"/>
 <wire x1="226.06" y1="25.4" x2="220.98" y2="25.4" width="0.1524" layer="91"/>
 </segment>
@@
 <pinref part="U1" gate="G$1" pin="*D9"/>
 <wire x1="147.32" y1="157.48" x2="157.48" y2="157.48" width="0.1524" layer="91"/>
-<pinref part="J5-D1" gate="G$1" pin="SHIELD2"/>
+<pinref part="J5-D9" gate="G$1" pin="SHIELD2"/>
 <wire x1="226.06" y1="35.56" x2="203.2" y2="35.56" width="0.1524" layer="91"/>
 </segment>
@@
 <wire x1="101.6" y1="71.12" x2="101.6" y2="68.58" width="0.1524" layer="91"/>
 </segment>
-</net>
+<segment>
+<pinref part="U2" gate="G$1" pin="OUT"/>
+<pinref part="C5" gate="G$1" pin="+"/>
+<wire x1="55.88" y1="152.4" x2="63.5" y2="152.4" width="0.1524" layer="91"/>
+<wire x1="63.5" y1="152.4" x2="63.5" y2="149.86" width="0.1524" layer="91"/>
+<wire x1="63.5" y1="152.4" x2="71.12" y2="152.4" width="0.1524" layer="91"/>
+<junction x="63.5" y="152.4"/>
+<pinref part="SUPPLY15" gate="G$1" pin="3.3V"/>
+</segment>
+</net>
