File: boards/basic/imwiser-basic-v01.sch (EAGLE design)
At the start: 42 parts, among them J1-A2 PJ-313-SPAD, J2-A3 PJ-313-SPAD, J3-A4 PJ-313-SPAD, J4-A5 PJ-313-SPAD, J5-D9 PJ-313-SPAD, J6-D6 PJ-313-SPAD, J7-D5 PJ-313-SPAD, J8-D3 PJ-313-SPAD, Q1 MOSFET-NCHANNEL2N7000, Q2 MOSFET-NCHANNEL2N7000, U1 ARDUINO_SHIELDNO_SILK

Commit message: Organized files, left organize cam jobs and libraries
Parts:
- removed C2: 10uF, SparkFun-Capacitors:10UF-25V-20%(PTH)
- removed C3, C4: 100nF, SparkFun-Capacitors:CAPPTH
- removed C5: 47uF, SparkFun-Capacitors:10UF-25V-20%(PTH)
- removed CURRENT0, CURRENT1, PROG: 2PIN, SparkFun-Connectors:M02PTH
- removed D1, D2: 1N5817, adafruit:SCHOTTKY-DIODEDO41-7
- removed ESP: ESP01, esp8266-modules:ESP01
- removed ESP-CON: 3PIN, SparkFun-Connectors:M03PTH
- removed J1-A2, J2-A3, J3-A4, J4-A5, J5-D9, J7-D5, J8-D3: PJ-313-SPAD, salvador-parts:PJ-313-SPAD
- removed Q1, Q2: MOSFET-NCHANNEL2N7000, SparkFun-DiscreteSemi:MOSFET-NCHANNEL2N7000
- removed R10, R11, R12, R9: 2.2K, resistor:R-US_0207/10
- removed R13, R14, R15: 10K, resistor:R-US_0207/10
- removed R5: 64, resistor:R-US_0207/10
- removed R6: 82, resistor:R-US_0207/10
- removed R7, R8: 470K, resistor:R-US_0207/10
- removed REG: 78D33, salvador-parts-imported:V_REG_78XXSINK
- removed S1: SWITCH-MOMENTARY-2PTH, salvador-parts-imported2:SWITCH-MOMENTARY-2PTH
- added CURRENT: (no value), SparkFun-Connectors:M02PTH
- added J1-A3, J2-A2, J3-A1, J4-D3, J5-D5: PJ-313-SPAD, salvador-parts:PJ-313-SPAD
- C1: value 10uF -> (none)
- D2-3, DOUT: value 3PIN -> (none)
Connections:
- net N$14 renamed D2
- net N$8 renamed OPTION-D2-3
- removed net 3.3V: C5.+, ESP.VCC, Q1.G, Q2.G, R11.2, R13.2, R14.2, R15.2, R9.2, REG.OUT
- removed net A4: J3-A4.SHIELD1, U1.A4
- removed net A5: J4-A5.SHIELD1, U1.A5
- removed net BURDEN-C1: C1.+, CURRENT1.1, R1.1, R2.1, R3.1, R4.2
- removed net CH-PD: C3.1, ESP.CH_PD, R14.1
- removed net D9: J5-D9.SHIELD2, U1.*D9
- removed net DTR: D2.C, ESP-CON.3
- removed net ESP-RX: ESP.RXD, Q2.S, R11.1
- removed net ESP-TX: ESP.TXD, Q1.S, R9.1
- removed net GPIO0: D1.A, ESP.GPIO0, PROG.1, R13.1
- removed net N$16: J5-D9.L2, J6-D6.L1
- removed net RST: ESP.RST, R15.1, S1.2
- removed net U$1: C3.2, D1.C, D2.A
- removed net UC-RX: ESP-CON.1, Q1.D, R10.1, U1.RX
- removed net UC-TX: ESP-CON.2, Q2.D, R12.1, U1.TX
- net A0: now also CURRENT.2, R1.2, R2.2; no longer CURRENT0.2, R5.2, R6.2
- net A1: now also J3-A1.SHIELD1; no longer CURRENT1.2, R1.2, R2.2
- net A2: now also J2-A2.SHIELD1; no longer J1-A2.SHIELD1
- net A3: now also J1-A3.SHIELD1; no longer J2-A3.SHIELD1
- net BURDEN-C0: now also C1.+, CURRENT.1, R1.1, R2.1, R3.1, R4.2; no longer C2.+, CURRENT0.1, R5.1, R6.1, R7.1, R8.2
- net D3: now also J4-D3.SHIELD1; no longer J8-D3.SHIELD1
- net D5: now also J5-D5.SHIELD1; no longer J7-D5.SHIELD2
- net GND: now also J1-A3.R, J2-A2.R, J3-A1.R, J4-D3.R, J5-D5.R; no longer C2.-, C4.2, C5.-, ESP.GND, J1-A2.R, J2-A3.R, J3-A4.R, J4-A5.R, J5-D9.R, J7-D5.R, J8-D3.R, PROG.2, R8.1, REG.GND, S1.1, S1.P$1
- net N$1: now also J1-A3.L2, J2-A2.L1; no longer J2-A3.L1, J3-A4.L2
- net N$2: now also J2-A2.L2, J3-A1.L1; no longer J1-A2.L1, J2-A3.L2
- net N$7: now also J4-D3.L1, J5-D5.L2; no longer J7-D5.L2, J8-D3.L1
- net N$9: now also J5-D5.L1; no longer J7-D5.L1
- net VCC: now also J1-A3.L1, J4-D3.L2; no longer C4.1, J3-A4.L1, J4-A5.L2, J8-D3.L2, R10.2, R12.2, R7.2, REG.IN
Other:
- note added: "DIGITAL SENSORS/ACTUATORS"
- note removed: "3.3V POWER SUPPLY"
- note removed: "5V - 3.3V BIDIRECTIONAL UART CONVERTER"
- note removed: "DIGITAL SENSORS"
- note removed: "ESP8266"
- note removed: "ESP8266 CONNECTOR"
- note removed: "ESP8266 FTDI-AUTORESET"
- moved on the sheet: C1, D2-3, DOUT, J6-D6, R1, R2, R3, R4, U1
