File: boards/esp-extended/imwiser-esp-v01.brd (EAGLE design)
At the start: 53.1 x 84.2 mm, 42 parts, among them J1-A2 PJ-313-SPAD, J2-A3 PJ-313-SPAD, J3-A4 PJ-313-SPAD, J4-A5 PJ-313-SPAD, J5-D9 PJ-313-SPAD, J6-D6 PJ-313-SPAD, J7-D5 PJ-313-SPAD, J8-D3 PJ-313-SPAD, Q1 MOSFET-NCHANNEL2N7000, Q2 MOSFET-NCHANNEL2N7000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

Commit message: Finished version 0.1 of imwiser for ESP
Parts:
- added ESP-EN: DPDT-GENERIC-SWITCH-7X7MM, salvador-parts:DPDT-PTH-7*7MM
- C4: value 100nF -> 0.33uF
- moved PROG 0.57 mm to (12.8, 56.4), turned to 0 degrees
- renumbered S1 to RESET
Connections:
- new net ESP-RX-5V: ESP-EN.3-IN1, Q2.3, R12.1
- new net ESP-TX-5V: ESP-EN.4-IN2, Q1.3, R10.1
- new net PROG-RX: ESP-CON.1, ESP-EN.2-OUT2-A
- new net PROG-TX: ESP-CON.2, ESP-EN.1-OUT1-A
- net UC-RX: now also ESP-EN.6-OUT2-B; no longer ESP-CON.1, Q1.3, R10.1
- net UC-TX: now also ESP-EN.5-OUT1-B; no longer ESP-CON.2, Q2.3, R12.1
Routing:
- net UC-TX: track 56.4 -> 11.2 mm
- net UC-RX: track 59.1 -> 17.6 mm
- net ESP-TX-5V: track 0.00 -> 39.1 mm
- net ESP-RX-5V: track 0.00 -> 34.5 mm
- net PROG-RX: track 0.00 -> 15.9 mm
- net PROG-TX: track 0.00 -> 12.1 mm
- net GPIO0: track 51.0 -> 59.1 mm
- net GND: track 304.9 -> 301.3 mm
